File: RoboSphere/RoboSphere.kicad_sch (KiCad schematic)
At the start: 20 parts, among them SW1 SW_Push, U1 RASPBERRY_PI_ZERO_2_W, U2 DRV8833PWP, U3 ADS1115IDGS, U5 L7806

Commit message: Finished Version 1
Parts:
- removed 10uF1, 10uF2: C, symbol Device:C
- removed AOUT1, AOUT2, BOUT1, BOUT2: Conn_01x03_Pin, Connector_PinHeader_2.54mm:PinHeader_1x03_P2.54mm_Vertical_SMD_Pin1Left, symbol Connector:Conn_01x03_Pin
- removed C3: 2.2uF, Capacitor_SMD:C_0805_2012Metric, symbol Device:C
- removed D1: Red, symbol Device:LED
- removed D2: Green, symbol Device:LED
- removed R1: 500 Ohm, symbol Device:R
- removed R2: 420 Ohm, symbol Device:R
- removed U2: DRV8833PWP, Package_SO:HTSSOP-16-1EP_4.4x5mm_P0.65mm_EP3.4x5mm_Mask2.46x2.31mm_ThermalVias, symbol Driver_Motor:DRV8833PWP
- removed U5: L7806, symbol Regulator_Linear:L7905
- added M1, M2: Motor_DC, symbol Motor:Motor_DC
- added Q1, Q2: BC557, Package_TO_SOT_THT:TO-92_Inline, symbol Transistor_BJT:BC557
- added U2: L7806, symbol Regulator_Linear:L7806
- 3350mAh2, 3350mAh3: value 3.6V -> 3.7V
- C1: value 0.01uF -> C; footprint Capacitor_SMD:C_0805_2012Metric -> (none)
- C2: value 10uF -> C; footprint Capacitor_SMD:C_0805_2012Metric -> (none)
Connections:
- net +6V: now also C2.2, U2.3 (OUT); no longer C1.1, C2.1, U1.2 (5V_2), U1.4 (5V_4)
- net GND: now also C1.1, C2.1, U3.1 (ADDR), U2.2 (GND); no longer C2.2, U1.14 (GND_14), U1.20 (GND_20), U1.25 (GND_25), U1.30 (GND_30), U1.34 (GND_34), U1.39 (GND_39), U1.6 (GND_6), U1.9 (GND_9)
- net at SW1.2, U3.4 (AIN0): now also C1.2, U2.1 (IN)
- net at U1.12 (GPIO18/GPIO_GEN1): now also Q1.2 (B)
- net at U1.29 (GPIO5): now also U3.2 (ALERT/RDY)
- net at U1.32 (GPIO12): now also Q2.2 (B)
- new net: Q1.1 (C), Q2.1 (C), U1.4 (5V_4)
- new net: M1.2 (-), M2.2 (-), U1.9 (GND_9)
- new net: M1.1 (+), Q1.3 (E)
- new net: M2.1 (+), Q2.3 (E)
Other:
- moved on the sheet: 3350mAh2, 3350mAh3, SW1, U1

Commit message: Updated schematic with placement organization
Parts:
- removed Q1, Q2: BC557, Package_TO_SOT_THT:TO-92_Inline, symbol Transistor_BJT:BC557
- removed U3: ADS1115IDGS, Package_SO:TSSOP-10_3x3mm_P0.5mm, symbol Analog_ADC:ADS1115IDGS
- added U4: L293D, Package_DIP:DIP-16_W7.62mm, symbol Driver_Motor:L293D
- added U5: ADS1115 1085, 1085:MODULE_1085, symbol 1085:1085
- C1, C2: footprint (none) -> Capacitor_THT:C_Disc_D3.0mm_W1.6mm_P2.50mm
- M1, M2: footprint (none) -> Motors:Vybronics_VZ30C1T8219732L
- SW1: footprint (none) -> Button_Switch_THT:SW_PUSH_6mm
- U1: footprint RASPBERRY_PI_ZERO_2_W:MODULE_RASPBERRY_PI_ZERO_2_W -> Module:Raspberry_Pi_Zero_Socketed_THT_FaceDown_MountingHoles
- U2: footprint (none) -> L7806CV:TO255P1020X450X1968-3B
Connections:
- net GND: now also U4.12 (GND), U4.13 (GND), U4.4 (GND), U4.5 (GND), U5.JP2_2 (GND), U5.JP2_5 (ADDR)
- net at U1.1 (3V3_1): now also U5.JP2_1 (VIN)
- net at U1.16 (GPIO23/GPIO_GEN4): now also U4.2 (1A)
- net at U1.18 (GPIO24/GPIO_GEN5): now also U4.7 (2A)
- net at U1.24 (GPIO8/SPI_~{CE0}): now also U4.10 (3A)
- net at U1.26 (GPIO7/SPI_~{CE1}): now also U4.15 (4A)
- net at U1.29 (GPIO5): now also U5.JP2_6 (ALRT)
- net at U1.3 (GPIO2/SDA1): now also U5.JP2_4 (SDA)
- net at U1.33 (GPIO13): now also U4.9 (EN3,4)
- net at U1.35 (GPIO19): now also U4.1 (EN1,2)
- net at U1.5 (GPIO3/SCL): now also U5.JP2_3 (SCL)
- net +7.5V: now reaches C1.2, SW1.2, U2.1 (IN)
- net +7.5V: now also U4.16 (VCC1), U4.8 (VCC2), U5.JP1_5 (A0)
- net at M1.1 (+): now also U4.11 (3Y)
- net at M2.1 (+): now also U4.3 (1Y)
- new net: M1.2 (-), U4.14 (4Y)
- new net: M2.2 (-), U4.6 (2Y)
- new net: U5.SH1 (SHIELD), U5.SH2 (SHIELD), U5.SH3 (SHIELD), U5.SH4 (SHIELD)
- now unconnected: U1.9 (GND_9)
Other:
- moved on the sheet: M1
